File: mcp1824bo.sch (EAGLE design)
At the start: 20 parts, among them J1 M02PTH, J2 M02PTH, J3 M02PTH, J4 10118194-0001LF, U4 MCP1824T-ADJE/OT

Commit message: replace SHDN jumper with a slide switch
Parts:
- removed J3: M02PTH, C3-Connector:M02PTH
- added SW1: CL-SB-12A-01, C3-Switches:CL-SB-12A-01
Connections:
- net GND: now also SW1.1
- net SHDN: now also SW1.2; no longer J3.2
- net VIN: now also SW1.3; no longer J3.1
Changed lines of the file:
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@@
 <attributes>
 <attribute name="PART_NUM" value="MCP1824BO"/>
-<attribute name="REV" value="A"/>
+<attribute name="REV" value="B"/>
 <attribute name="TITLE" value="MCP1824-ADJ Breakout"/>
 </attributes>
@@
 <part name="J1" library="C3-Connector" deviceset="M02" device="PTH"/>
 <part name="J2" library="C3-Connector" deviceset="M02" device="PTH"/>
-<part name="J3" library="C3-Connector" deviceset="M02" device="PTH"/>
 <part name="J4" library="C3-Connector" deviceset="M05" device="USB-MICRO" value="10118194-0001LF"/>
 <part name="D1" library="C3-Comchip" deviceset="CZRB*?" device="B-HF" technology="5338"/>
@@
 <part name="U$4" library="C3-General" deviceset="VOUT" device=""/>
 <part name="U$3" library="C3-General" deviceset="VOUT" device=""/>
+<part name="SW1" library="C3-Switches" deviceset="CL-SB-12?-*" device="A" technology="01"/>
 </parts>
 <sheets>
@@
 <instance part="J1" gate="G" x="71.12" y="142.24"/>
 <instance part="J2" gate="G" x="200.66" y="144.78" rot="R180"/>
-<instance part="J3" gate="G" x="91.44" y="127"/>
 <instance part="J4" gate="G$1" x="71.12" y="106.68"/>
 <instance part="D1" gate="A" x="104.14" y="91.44" rot="R90"/>
@@
 <instance part="U$4" gate="A" x="193.04" y="149.86"/>
 <instance part="U$3" gate="A" x="177.8" y="160.02"/>
+<instance part="SW1" gate="A" x="88.9" y="129.54" rot="R90"/>
 </instances>
 <busses>
@@
 <pinref part="C9" gate="A" pin="1"/>
 <pinref part="GND" gate="1" pin="GND"/>
-<wire x1="111.76" y1="134.62" x2="111.76" y2="111.76" width="0.1524" layer="91"/>
+<wire x1="111.76" y1="134.62" x2="111.76" y2="124.46" width="0.1524" layer="91"/>
 <pinref part="J4" gate="G$1" pin="5"/>
+<wire x1="111.76" y1="124.46" x2="111.76" y2="111.76" width="0.1524" layer="91"/>
 <wire x1="111.76" y1="111.76" x2="111.76" y2="88.9" width="0.1524" layer="91"/>
 <wire x1="111.76" y1="88.9" x2="111.76" y2="83.82" width="0.1524" layer="91"/>
@@
 <wire x1="104.14" y1="88.9" x2="111.76" y2="88.9" width="0.1524" layer="91"/>
 <junction x="111.76" y="88.9"/>
+<pinref part="SW1" gate="A" pin="1"/>
+<wire x1="99.06" y1="124.46" x2="111.76" y2="124.46" width="0.1524" layer="91"/>
+<junction x="111.76" y="124.46"/>
 </segment>
 <segment>
@@
 <wire x1="121.92" y1="129.54" x2="121.92" y2="109.22" width="0.1524" layer="91"/>
 <wire x1="121.92" y1="109.22" x2="127" y2="109.22" width="0.1524" layer="91"/>
-<pinref part="J3" gate="G" pin="2"/>
 <wire x1="99.06" y1="129.54" x2="116.84" y2="129.54" width="0.1524" layer="91"/>
 <junction x="121.92" y="129.54"/>
@@
 <wire x1="116.84" y1="93.98" x2="116.84" y2="129.54" width="0.1524" layer="91"/>
 <junction x="116.84" y="129.54"/>
+<pinref part="SW1" gate="A" pin="2"/>
 </segment>
 </net>
@@
 <pinref part="J1" gate="G" pin="2"/>
 <wire x1="78.74" y1="144.78" x2="104.14" y2="144.78" width="0.1524" layer="91"/>
-<pinref part="J3" gate="G" pin="1"/>
 <wire x1="104.14" y1="144.78" x2="111.76" y2="144.78" width="0.1524" layer="91"/>
-<wire x1="99.06" y1="127" x2="104.14" y2="127" width="0.1524" layer="91"/>
-<wire x1="104.14" y1="127" x2="104.14" y2="144.78" width="0.1524" layer="91"/>
 <junction x="104.14" y="144.78"/>
 <pinref part="U$1" gate="A" pin="VIN"/>
@@
 <wire x1="93.98" y1="101.6" x2="104.14" y2="101.6" width="0.1524" layer="91"/>
 <wire x1="104.14" y1="101.6" x2="104.14" y2="99.06" width="0.1524" layer="91"/>
-<wire x1="104.14" y1="127" x2="104.14" y2="101.6" width="0.1524" layer="91"/>
-<junction x="104.14" y="127"/>
+<wire x1="104.14" y1="144.78" x2="104.14" y2="134.62" width="0.1524" layer="91"/>
 <junction x="104.14" y="101.6"/>
 <pinref part="R3" gate="A" pin="1"/>
+<wire x1="104.14" y1="134.62" x2="104.14" y2="101.6" width="0.1524" layer="91"/>
 <wire x1="104.14" y1="162.56" x2="106.68" y2="162.56" width="0.1524" layer="91"/>
 <junction x="104.14" y="162.56"/>
-</segment>
-</net>
+<pinref part="SW1" gate="A" pin="3"/>
+<wire x1="99.06" y1="134.62" x2="104.14" y2="134.62" width="0.1524" layer="91"/>
+<junction x="104.14" y="134.62"/>
+</segment>
+</net>
